File: Kicad/EchoLink/EchoLink.kicad_pcb (KiCad board)
At the start: 4 copper layers, 50.8 x 101.6 mm, 75 parts, among them J1 142-0701-801, J3 Conn_01x07_Pin, J5 Conn_01x07_Pin, J7 Conn_01x06_Pin, J8 Conn_01x05_Pin, SW1 SW_Push, SW2 SW_Push, U1 STM32L433CCT6, U2 E22-400M33S, U3 ISOW1044

Commit message: wip: pcb components
Parts:
- moved U2 190.2 mm to (119.5, 109.0), turned to 90 degrees
- moved J1 188.0 mm to (113.8, 66.7)
- moved C27 183.1 mm to (119.5, 8.54), turned to 180 degrees
- moved C26 181.5 mm to (119.5, 11.1), turned to 180 degrees
- moved C25 180.0 mm to (119.5, 13.6), turned to 180 degrees
- moved C17 179.4 mm to (123.0, 99.7)
- moved C23 177.4 mm to (119.5, 18.6), turned to 180 degrees
- moved R14 173.8 mm to (113.2, 4.99), turned to 90 degrees
- moved C21 172.2 mm to (102.4, 5.00), turned to 90 degrees
- moved R11 171.9 mm to (123.1, 95.9)
- moved R12 171.5 mm to (123.0, 101.3)
- moved R10 171.3 mm to (123.0, 98.1), turned to 180 degrees
- moved C20 169.8 mm to (100.8, 5.00), turned to 90 degrees
- moved C19 167.4 mm to (99.2, 5.00), turned to 90 degrees
- moved R13 166.7 mm to (106.5, 5.00), turned to 90 degrees
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
Commit message: wip: positionning and polygon planes
Parts:
- moved H2 149.3 mm to (47.0, 3.81)
- moved C12 126.2 mm to (46.4, 10.3), turned to 90 degrees
- moved J3 125.7 mm to (45.5, 36.6), turned to 180 degrees
- moved R17 124.5 mm to (12.8, 49.5), turned to 180 degrees
- moved R8 123.0 mm to (46.4, 13.4), turned to 90 degrees
- moved D2 120.5 mm to (9.65, 49.5)
- moved SW1 119.8 mm to (42.3, 11.7), turned to -90 degrees
- moved H4 119.4 mm to (47.0, 97.8)
- moved R6 118.3 mm to (45.7, 16.5), turned to 90 degrees
- moved D1 115.3 mm to (43.0, 16.9), turned to 0 degrees
- moved C1 112.1 mm to (45.0, 46.8), turned to 0 degrees
- moved H1 111.9 mm to (3.81, 3.81)
- moved R1 111.2 mm to (41.8, 46.8), turned to 0 degrees
- moved JP1 108.7 mm to (41.5, 49.8)
- moved R5 108.7 mm to (45.9, 49.6)
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Connections:
- H1 pad 1: (no net) -> GND
- H2 pad 1: (no net) -> GND
- H3 pad 1: (no net) -> GND
- H4 pad 1: (no net) -> GND
- U2 pad 0: (no net) -> GND
Routing:
- net Net-(U2-ANT): track 0.00 -> 15.6 mm
- net GND: vias 0 -> 127
- added copper zone on B.Cu, net GND
- added copper zone on F.Cu, net GND
Other:
- outline, holes or cut-outs redrawn

Commit message: wip: add hse crystal and update stm32 project (clock 80MHz and 500kbps CAN)
Parts:
- removed J3: Conn_01x07_Pin, Connector_PinHeader_2.54mm:PinHeader_1x07_P2.54mm_Vertical
- added C10: 22pF, Capacitor_SMD:C_0603_1608Metric, F.Cu at (84.3, 67.0)
- added C14: 22pF, Capacitor_SMD:C_0603_1608Metric, F.Cu at (84.3, 69.6)
- added R10: 10R, Resistor_SMD:R_0603_1608Metric, F.Cu at (84.3, 72.1)
- added Y1: WE-XTAL_HC49, EchoLink_Lib:WE-XTAL_HC49, F.Cu at (88.7, 62.6)
- moved C15 31.9 mm to (65.3, 28.7)
- moved C8 31.9 mm to (58.1, 28.9)
- moved FB1 31.9 mm to (62.7, 28.2)
- moved C11 31.9 mm to (59.8, 28.6)
- moved R2 21.9 mm to (62.9, 38.2)
- moved JP1 21.9 mm to (60.2, 38.4)
- moved R4 21.9 mm to (64.6, 38.2)
- moved C2 19.7 mm to (63.3, 54.2)
- moved SW2 19.7 mm to (61.7, 50.0)
- moved R5 19.7 mm to (60.1, 54.2)
- renumbered C12 to C1, C9 to C11, C10 to C12, C11 to C13, C13 to C15, C14 to C16, C15 to C17, C16 to C18, C17 to C19, C1 to C2, C18 to C20, C19 to C21, C20 to C22, C21 to C23, C22 to C24, C23 to C25, C24 to C26, C25 to C27, C26 to C28, C27 to C29, C2 to C3, C3 to C4, C4 to C5, C5 to C6, C6 to C7, C7 to C8, C8 to C9, R6 to R1, R10 to R11, R11 to R12, R12 to R13, R13 to R14, R14 to R15, R15 to R16, R16 to R17, R17 to R18, R4 to R2, R8 to R3, R5 to R4, R1 to R5, R2 to R6, R3 to R7, R7 to R8
Connections:
- H1 pad 1: GND -> (no net)
- H2 pad 1: GND -> (no net)
- H3 pad 1: GND -> (no net)
- H4 pad 1: GND -> (no net)
- U1 pad 4: EXTEND_IO1 -> unconnected-(U1-PC15-OSC32_OUT-Pad4)
- U1 pad 5: EXTEND_IO2 -> OSC_IN
- U1 pad 6: EXTEND_IO3 -> OSC_OUT
- U2 pad 0: GND -> (no net)
